File: DSPFX.kicad_sch (KiCad schematic)
At the start: 116 parts, among them J10 Conn_02x05_Odd_Even, J101 AudioJack2, J102 AudioJack2, J103 AudioJack2, J104 AudioJack2, J105 Conn_02x04_Odd_Even, J106 AudioJack2, J107 AudioJack2, J108 AudioJack2, J109 AudioJack2, J110 AudioJack2, J111 AudioJack2, J112 AudioJack2, J113 AudioJack2_SwitchT, J114 Conn_02x04_Odd_Even, J115 Conn_01x04_Pin, J116 Conn_01x04_Pin, J117 Conn_01x04_Pin, J118 Conn_01x04_Pin, J119 Conn_01x04_Pin, J120 Conn_01x04_Pin, J121 Conn_01x03_Pin, J122 Conn_01x04_Pin, J123 Conn_01x02_Pin, J124 Conn_01x02_Pin, J125 Conn_01x03_Pin, J126 Conn_01x04_Pin, J127 Conn_01x04_Pin, J128 Conn_01x04_Pin, Q101 BC847, Q102 BC847, Q103 BC847, Q104 BC847, SW101 SW_Push, SW102 SW_Push, U101 TL074, U102 MCP6004, U104 TL072, U105 7Segment, U106 LM337_SOT223, U107 DSP32-CORE

Commit message: Swapped LEDs and Potentiometer parity issue
Connections:
- net LED2: now also D104.2 (A); no longer D107.2 (A)
- net LED3: now also D107.2 (A); no longer D104.2 (A)
- net LEDN2: now also D104.1 (K); no longer D107.1 (K)
- net LEDN3: now also D107.1 (K); no longer D104.1 (K)
Other:
- moved on the sheet: D104, D107
